Commit message: Update my_robot.xacro

File: my_robot/urdf/my_robot.xacro (robot description, xacro)
@@ -22,5 +22,5 @@
       <origin xyz="0 0 0" rpy=" 0 0 0"/>
       <geometry>
-        <box size=".4 .2 .1"/>
+        <cylinder radius="0.4" length="0.1"/>
       </geometry>
     </collision>
@@ -28,5 +28,5 @@
       <origin xyz="0 0 0" rpy=" 0 0 0"/>
       <geometry>
-        <box size=".4 .2 .1"/>
+        <cylinder radius="0.4" length="0.1"/>
       </geometry>
     </visual>
@@ -86,5 +86,5 @@
   </link>
   <joint type="continuous" name="left_wheel_hinge">
-    <origin xyz="0 0.15 0" rpy="0 0 0"/>
+    <origin xyz="0 0.25 0" rpy="0 0 0"/>
     <child link="left_wheel"/>
     <parent link="chassis"/>
@@ -118,5 +118,5 @@
   </link>
   <joint type="continuous" name="right_wheel_hinge">
-    <origin xyz="0 -0.15 0" rpy="0 0 0"/>
+    <origin xyz="0 -0.25 0" rpy="0 0 0"/>
     <child link="right_wheel"/>
     <parent link="chassis"/>

Commit message: Change the shape of mobile robot base from cube to cylinder.

File: my_robot/urdf/my_robot.xacro (robot description, xacro)
@@ -22,5 +22,5 @@
       <origin xyz="0 0 0" rpy=" 0 0 0"/>
       <geometry>
-        <cylinder radius="0.4" length="0.1"/>
+        <cylinder radius="0.2" length="0.1"/>
       </geometry>
     </collision>
@@ -28,5 +28,5 @@
       <origin xyz="0 0 0" rpy=" 0 0 0"/>
       <geometry>
-        <cylinder radius="0.4" length="0.1"/>
+        <cylinder radius="0.2" length="0.1"/>
       </geometry>
     </visual>

Commit message: Upgrade sensor to RGBD camera - Add optical camera link in .xacro - Replace old RGB camera plugin with Kinect RGBD camera

File: my_robot/urdf/my_robot.xacro (robot description, xacro)
@@ -190,3 +190,10 @@
     <child link="hokuyo"/>
   </joint>
+  <joint name="camera_optical_joint" type="fixed">
+    <origin xyz="0 0 0" rpy="0 0 0"/>
+    <parent link="camera"/>
+    <child link="camera_link_optical"/>
+  </joint>
+  <link name="camera_link_optical">
+  </link>
 </robot>

Commit message: Change world layout - Use smaller world to speed up mapping process

File: my_robot/urdf/my_robot.xacro (robot description, xacro)
@@ -191,5 +191,5 @@
   </joint>
   <joint name="camera_optical_joint" type="fixed">
-    <origin xyz="0 0 0" rpy="0 0 0"/>
+    <origin xyz="0 0 0" rpy="-1.5707 0 -1.5707"/>
     <parent link="camera"/>
     <child link="camera_link_optical"/>
